File: PCB/Detector_rev2/Detector_rev2.sch (KiCad schematic (older format))
At the start: 60 parts, among them J2 Conn_01x03_Male, J3 Conn_Coaxial, U1 N-jfet_dual, U2 N-jfet_dual, U3 LM6171D, U4 LM6171D, U5 LT6657BHMS8-5, U6 LT1995, U7 DMMT3904

Commit message: garberdata output
Parts:
- J1: renamed from J?; footprint Connector_JST:JST_XH_S3B-XH-A-1_1x03_P2.50mm_Horizontal -> Detector_rev2:input
- J2: footprint Connector_JST:JST_XH_S3B-XH-A-1_1x03_P2.50mm_Horizontal -> Detector_rev2:JST-XH_S3B
Changed lines of the file:
@@
 F 0 "J2" H 5208 1481 50  0000 C CNN
 F 1 "Conn_01x03_Male" H 5208 1390 50  0000 C CNN
-F 2 "Connector_JST:JST_XH_S3B-XH-A-1_1x03_P2.50mm_Horizontal" H 5100 1200 50  0001 C CNN
+F 2 "Detector_rev2:JST-XH_S3B" H 5100 1200 50  0001 C CNN
 F 3 "~" H 5100 1200 50  0001 C CNN
 	1    5100 1200
@@
 $EndComp
 $Comp
-L Connector:Conn_01x03_Male J?
+L Connector:Conn_01x03_Male J1
 U 1 1 5EE8C568
 P 1500 4200
-F 0 "J?" H 1608 4481 50  0000 C CNN
+F 0 "J1" H 1608 4481 50  0000 C CNN
 F 1 "Conn_01x03_Male" H 1608 4390 50  0000 C CNN
-F 2 "Connector_JST:JST_XH_S3B-XH-A-1_1x03_P2.50mm_Horizontal" H 1500 4200 50  0001 C CNN
+F 2 "Detector_rev2:input" H 1500 4200 50  0001 C CNN
 F 3 "~" H 1500 4200 50  0001 C CNN
 	1    1500 4200
@@
 	1900 5450 2800 5450
 $Comp
-L power:GND #PWR?
+L power:GND #PWR0111
 U 1 1 5EE9DC3B
 P 2600 4200
-F 0 "#PWR?" H 2600 3950 50  0001 C CNN
+F 0 "#PWR0111" H 2600 3950 50  0001 C CNN
 F 1 "GND" H 2605 4027 50  0000 C CNN
 F 2 "" H 2600 4200 50  0001 C CNN
