File: PCB/Detector_rev2/_autosave-Detector_rev2.kicad_pcb (KiCad board)
At the start: 2 copper layers, 51.4 x 44.4 mm, 56 parts, among them J1 Conn_01x03_Male, J2 Conn_01x03_Male, J3 Conn_Coaxial, U1 N-jfet_dual, U2 N-jfet_dual, U3 LM6171D, U4 LM6171D, U5 LT6657BHMS8-5, U6 LT1995, U7 DMMT3904

Commit message: input terminal adjust
Parts:
- moved J1 0.76 mm to (52.6, 68.3)
Routing:
- net GND: vias 215 -> 216
- net (no net): vias 0 -> 1
Changed lines of the file:
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@@
-(kicad_pcb (version 20171130) (host pcbnew "(5.1.0-0)")
+(kicad_pcb (version 20171130) (host pcbnew "(5.1.5)-3")
   (general
     (thickness 1.6)
     (drawings 4)
-    (tracks 541)
+    (tracks 543)
     (zones 0)
     (modules 56)
@@
   )
   (setup
-    (last_trace_width 0.25)
+    (last_trace_width 0.8)
     (user_trace_width 0.5)
     (user_trace_width 0.8)
     (user_trace_width 1.25)
     (trace_clearance 0.2)
-    (zone_clearance 0.2)
+    (zone_clearance 0.1)
     (zone_45_only no)
     (trace_min 0.2)
@@
   )
   (module Detector_rev2:input (layer F.Cu)
-    (at 53.34 68.326)
-    (fp_text reference J1 (at 5.08 -5.08) (layer F.SilkS)
+    (at 52.578 68.2625)
+    (fp_text reference J1 (at 1.27 -4.699) (layer F.SilkS)
       (effects (font (size 1 1) (thickness 0.15)))
     )
@@
     (tags resistor)
     (attr smd)
-    (fp_text reference R2 (at 0.7875 -1.27 90) (layer F.SilkS)
+    (fp_text reference R2 (at -0.1015 -1.397 90) (layer F.SilkS)
       (effects (font (size 1 1) (thickness 0.15)))
     )
@@
   (gr_line (start 50.165 87.63) (end 50.165 43.18) (layer Edge.Cuts) (width 0.1))
   (gr_line (start 101.6 87.63) (end 50.165 87.63) (layer Edge.Cuts) (width 0.1))
-  (via (at 54.864 68.326) (size 0.8) (drill 0.4) (layers F.Cu B.Cu) (net 1))
-  (via (at 53.848 68.326) (size 0.8) (drill 0.4) (layers F.Cu B.Cu) (net 1))
-  (via (at 52.832 68.326) (size 0.8) (drill 0.4) (layers F.Cu B.Cu) (net 1))
-  (via (at 52.07 68.834) (size 0.8) (drill 0.4) (layers F.Cu B.Cu) (net 1))
-  (via (at 52.07 67.818) (size 0.8) (drill 0.4) (layers F.Cu B.Cu) (net 1))
+  (via (at 82.55 74.93) (size 0.8) (drill 0.4) (layers F.Cu B.Cu) (net 0))
+  (via (at 82.55 72.39) (size 0.8) (drill 0.4) (layers F.Cu B.Cu) (net 1))
+  (via (at 53.848 68.2625) (size 0.8) (drill 0.4) (layers F.Cu B.Cu) (net 1))
+  (via (at 52.8955 68.2625) (size 0.8) (drill 0.4) (layers F.Cu B.Cu) (net 1))
+  (via (at 51.943 68.2625) (size 0.8) (drill 0.4) (layers F.Cu B.Cu) (net 1))
+  (via (at 51.181 68.7705) (size 0.8) (drill 0.4) (layers F.Cu B.Cu) (net 1))
+  (via (at 51.181 67.7545) (size 0.8) (drill 0.4) (layers F.Cu B.Cu) (net 1))
   (segment (start 67.31 56.388) (end 67.818 56.388) (width 0.8) (layer F.Cu) (net 1))
   (segment (start 69.342 54.864) (end 71.501 54.864) (width 0.8) (layer F.Cu) (net 1))
@@
   )
   (zone (net 1) (net_name GND) (layer F.Cu) (hatch edge 0.508)
-    (connect_pads (clearance 0.6))
-    (min_thickness 0.2)
-    (fill yes (arc_segments 32) (thermal_gap 0.508) (thermal_bridge_width 0.508))
-    (polygon
-      (pts
-        (xy 101.6 87.63) (xy 50.165 87.63) (xy 50.165 43.18) (xy 101.6 43.18)
-      )
-    )
-  )
-  (zone (net 1) (net_name GND) (layer F.Cu) (hatch edge 0.508)
     (priority 1)
     (connect_pads yes (clearance 0.2))
@@
       )
     )
+  )
+  (zone (net 1) (net_name GND) (layer F.Cu) (hatch edge 0.508)
+    (connect_pads (clearance 0.6))
+    (min_thickness 0.2)
+    (fill yes (arc_segments 32) (thermal_gap 0.508) (thermal_bridge_width 0.508))
+    (polygon
+      (pts
+        (xy 101.6 87.63) (xy 50.165 87.63) (xy 50.165 43.18) (xy 101.6 43.18)
+      )
+    )
+  )
+  (zone (net 1) (net_name GND) (layer F.Cu) (hatch edge 0.508)
+    (priority 2)
+    (connect_pads yes (clearance 0.1))
+    (min_thickness 0.2)
+    (fill yes (arc_segments 32) (thermal_gap 0.508) (thermal_bridge_width 0.508))
+    (polygon
+      (pts
+        (xy 59.055 67.818) (xy 59.055 68.707) (xy 53.7845 68.707) (xy 53.7845 67.818)
+      )
+    )

Commit message: garberdata output
Parts:
- J2: footprint Connector_JST:JST_XH_S3B-XH-A-1_1x03_P2.50mm_Horizontal -> Detector_rev2:JST-XH_S3B
- moved J2 2.56 mm to (93.2, 53.6)
- moved H4 0.72 mm to (52.8, 45.7)
- moved H3 0.64 mm to (98.3, 84.5)
- moved TP2 0.51 mm to (75.5, 65.0)
- moved H2 0.51 mm to (98.3, 45.7)
- moved J1 0.51 mm to (52.1, 68.3)
- moved H1 0.35 mm to (52.8, 84.5)
Routing:
- net GND: vias 216 -> 215
- net (no net): vias 1 -> 0
Other:
- board size 51.4 x 44.4 mm -> 52.1 x 45.1 mm
- rule solder_mask_min_width: 0.25 -> 0.001
- rule trace_min: 0.2 -> 0.01
