File: PCB/GradientDriver_rev2/GradientDriver.kicad_pcb (KiCad board)
At the start: 4 copper layers, 54.6 x 67.9 mm, 61 parts, among them J1 Conn_01x03, J2 Conn_Coaxial, J3 Conn_Coaxial, J4 Conn_Coaxial, U1 OP37GSZ-REEL7, U2 AD8603, U3 OPA548TG3, U4 OPA548TG3, U5 L7812, U6 L7912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

Commit message: GradDriver rev2 edit
Parts:
- moved C15 12.6 mm to (91.3, 78.2)
- moved C13 11.4 mm to (94.3, 74.1)
- moved U5 11.3 mm to (94.0, 64.1)
- moved C14 5.75 mm to (85.9, 74.1)
- moved U6 5.74 mm to (86.4, 64.1)
- moved C16 4.91 mm to (86.6, 82.7), turned to 270 degrees
- moved R11 2.82 mm to (93.5, 87.0)
- moved R1 2.05 mm to (93.5, 85.5)
- moved R5 2.05 mm to (97.3, 85.5)
- moved U1 2.05 mm to (91.2, 81.7)
- moved C20 1.75 mm to (108.2, 91.1), turned to 0 degrees
- moved TP6 1.66 mm to (102.0, 58.5)
- moved TP7 0.65 mm to (111.1, 58.5)
- moved R14 0.40 mm to (116.3, 94.9)
Connections:
- U6 pad 4: (no net) -> -15V
Routing:
- net -15V: track 62.2 -> 138.7 mm, vias 6 -> 18
- net +12VA: track 17.8 -> 55.1 mm, vias 5 -> 7
- net +15V: track 55.9 -> 86.1 mm, vias 7 -> 6
- net -12VA: track 15.6 -> 41.3 mm, vias 7 -> 8
- net GND: track 31.1 -> 20.2 mm, vias 138 -> 287
- net (no net): track 0.00 -> 6.30 mm, vias 12 -> 0
- net Net-(R1-Pad2): track 18.0 -> 13.0 mm
- net Net-(C2-Pad1): track 13.2 -> 15.4 mm
- net Net-(C2-Pad2): track 3.71 -> 5.20 mm
- net Net-(R11-Pad1): track 22.4 -> 21.0 mm
- net Net-(J4-Pad2): track 33.1 -> 33.7 mm
- added copper zone on F.Cu, net -15V
